File: maru-logic.kicad_pcb (KiCad board)
At the start: 2 copper layers, 223.5 x 116.8 mm, 464 parts, among them J101 USB-C, Q10001 2N7002, Q10101 2N7002, Q10201 2N7002, Q10301 2N7002, Q1701 2N7002, Q1801 2N7002, Q1901 2N7002, Q2001 2N7002, Q2101 2N7002, Q2201 2N7002, Q2301 2N7002, Q2401 2N7002, Q2501 2N7002, Q2601 2N7002, Q2701 2N7002, Q2801 2N7002, Q2901 2N7002, Q3001 2N7002, Q3201 2N7002, Q3301 2N7002, Q3401 2N7002, Q3501 2N7002, Q3601 2N7002, Q3701 2N7002, Q3801 2N7002, Q3901 2N7002, Q4001 2N7002, Q401 2N7002, Q4301 2N7002, Q4501 2N7002, Q4601 2N7002, Q4701 2N7002, Q4801 2N7002, Q4901 2N7002, Q5001 2N7002, Q5101 2N7002, Q5201 2N7002, Q5301 2N7002, Q5501 2N7002, Q5601 2N7002, Q5701 2N7002, Q5801 2N7002, Q5901 2N7002, Q6101 2N7002, Q6201 2N7002, Q6301 2N7002, Q6401 2N7002, Q6501 2N7002, Q6701 2N7002, Q6801 2N7002, Q6901 2N7002, Q7001 2N7002, Q7101 2N7002, Q7401 2N7002, Q7501 2N7002, Q7601 2N7002, Q7701 2N7002, Q7801 2N7002, Q8001 2N7002, Q8101 2N7002, Q8501 2N7002, Q8601 2N7002, Q8701 2N7002, Q8801 2N7002, Q8901 2N7002, Q9001 2N7002, Q9201 2N7002, Q9301 2N7002, Q9401 2N7002, Q9501 2N7002, Q9601 2N7002, Q9701 2N7002, Q9801 2N7002, Q9901 2N7002, SW1001 Push, SW1201 Push, SW1401 Push, SW1601 Push, SW301 Push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

Commit message: cloned
Parts:
- moved Q2501 358.2 mm to (402.6, 154.9)
- moved D2501 357.8 mm to (402.1, 160.0)
- moved R2502 355.0 mm to (403.6, 157.5)
- moved C2501 354.4 mm to (401.6, 157.5)
- moved R2501 353.7 mm to (401.6, 152.4)
- moved Q2201 353.3 mm to (417.8, 154.9)
- moved D2201 353.0 mm to (417.3, 160.0)
- moved R2202 350.2 mm to (418.8, 157.5)
- moved C2201 349.4 mm to (416.8, 157.5)
- moved R2201 348.6 mm to (416.8, 152.4)
- moved Q8701 330.1 mm to (392.4, 154.9)
- moved D8701 329.7 mm to (391.9, 160.0)
- moved R8702 326.9 mm to (393.4, 157.5)
- moved C8701 326.3 mm to (391.4, 157.5)
- moved R8701 325.5 mm to (391.4, 152.4)
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Routing:
- net VSS: track 105.7 -> 369.3 mm, vias 34 -> 107
- net /ALL_Y: track 0.00 -> 6.38 mm
- net /Chain OR_X/LINK4: track 0.00 -> 6.37 mm
- net /Chain OR_X/LINK3: track 0.00 -> 6.37 mm
- net /Chain OR_X/LINK1: track 0.00 -> 6.37 mm
- net /Chain OR_B/LINK3: track 0.00 -> 6.37 mm
- net /Chain OR_B/LINK1: track 0.00 -> 6.37 mm
- net /Chain NOT_X/LINK4: track 0.00 -> 6.37 mm
- net /Chain NOT_X/LINK3: track 0.00 -> 6.37 mm
- net /Chain NOT_X/LINK1: track 0.00 -> 6.37 mm
- net /Chain NOT_A/LINK4: track 0.00 -> 6.37 mm
- net /Chain NOT_A/LINK1: track 0.00 -> 6.37 mm
- net /Chain ALL_Y1/LINK4: track 0.00 -> 6.37 mm
- net /Chain ALL_Y1/LINK2: track 0.00 -> 6.37 mm
- net /Chain XOR_B/LINK3: track 0.00 -> 6.37 mm
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
Commit message: layout done, starting case
Parts:
- removed C8501, C8601, C8701, C8801, C8901, C9001, C9201, C9301, C9401, C9501, C9601, C9701: 1u, Capacitor_SMD:C_0402_1005Metric
- removed D8501, D8601, D8701, D8801, D8901, D9001, D9201, D9301, D9401, D9501, D9601, D9701: White, mark:LED_0603_1608Metric_no_silk
- removed Q8501, Q8601, Q8701, Q8801, Q8901, Q9001, Q9201, Q9301, Q9401, Q9501, Q9601, Q9701: 2N7002, Package_TO_SOT_SMD:SOT-23
- removed R8501, R8601, R8701, R8801, R8901, R9001, R9201, R9301, R9401, R9501, R9601, R9701: 100k, Resistor_SMD:R_0402_1005Metric
- removed R8502, R8602, R8702, R8802, R8902, R9002, R9202, R9302, R9402, R9502, R9602, R9702: 220, Resistor_SMD:R_0402_1005Metric
- moved C2201 294.7 mm to (157.2, 18.0), turned to -90 degrees
- moved R2201 293.2 mm to (157.2, 16.0), turned to -90 degrees
- moved Q2201 292.7 mm to (159.8, 16.8)
- moved R2202 292.7 mm to (160.8, 19.3)
- moved C2001 290.2 mm to (152.2, 18.0), turned to -90 degrees
- moved R2001 288.8 mm to (152.2, 16.0), turned to -90 degrees
- moved Q2001 288.3 mm to (154.7, 16.8)
- moved R2002 288.3 mm to (155.7, 19.3)
- moved C2301 285.8 mm to (147.1, 18.0), turned to -90 degrees
- moved C2401 285.8 mm to (162.3, 18.0), turned to -90 degrees
- moved R2301 284.3 mm to (147.1, 16.0), turned to -90 degrees
- moved R2401 284.3 mm to (162.3, 16.0), turned to -90 degrees
- moved Q2301 283.8 mm to (149.6, 16.8)
- moved Q2401 283.8 mm to (164.8, 16.8)
- moved R2302 283.8 mm to (150.6, 19.3)
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Routing:
- net VSS: track 369.3 -> 701.9 mm, vias 107 -> 201
- net /NOT_Y: track 6.37 -> 180.4 mm, vias 0 -> 4
- net /OR_Y: track 6.37 -> 175.7 mm, vias 0 -> 2
- net /ALL_X: track 0.00 -> 159.3 mm, vias 0 -> 2
- net /AND_Y: track 6.37 -> 116.8 mm, vias 0 -> 4
- net /BXA: track 19.9 -> 129.5 mm, vias 2 -> 8
- net /OR_A: track 7.64 -> 115.9 mm, vias 0 -> 4
- net VDD: track 301.2 -> 403.6 mm, vias 4 -> 31
- net /NOT_X: track 0.00 -> 101.8 mm, vias 0 -> 4
- net /XOR_A: track 15.9 -> 111.0 mm, vias 0 -> 8
- net /XOR_X: track 0.00 -> 93.6 mm, vias 0 -> 8
- net /XOR_Y: track 6.37 -> 98.1 mm, vias 0 -> 2
- net /AND_X: track 0.00 -> 89.1 mm, vias 0 -> 4
- net /OR_X: track 0.00 -> 87.8 mm, vias 0 -> 2
- net /XOR_B: track 18.8 -> 104.2 mm, vias 2 -> 8
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- added copper zone on B.Cu, net VDD
- added copper zone on F.Cu, net VSS
